Commit message: basic grippers added to the erdf files

File: src/ros2_control_demos/example_7/description/ros2_control/r6bot.ros2_control.xacro (robot description, xacro)
@@ -90,4 +90,26 @@
         <state_interface name="velocity"/>
       </joint>
+      <!-- ================= GRIPPER START ================= -->
+      <joint name="gripper_left_joint">
+        <command_interface name="position">
+          <param name="min">-0.03</param>
+          <param name="max">0.0</param>
+        </command_interface>
+        <state_interface name="position">
+          <param name="initial_value">0.0</param>
+        </state_interface>
+        <state_interface name="velocity"/>
+      </joint>
+      <joint name="gripper_right_joint">
+        <command_interface name="position">
+          <param name="min">0.0</param>
+          <param name="max">0.03</param>
+        </command_interface>
+        <state_interface name="position">
+          <param name="initial_value">0.0</param>
+        </state_interface>
+        <state_interface name="velocity"/>
+      </joint>
+      <!-- ================= GRIPPER END ================= -->
       <sensor name="tcp_fts_sensor">
         <state_interface name="force.x"/>

File: src/ros2_control_demos/ros2_control_demo_description/r6bot/urdf/r6bot_description.urdf.xacro (robot description, xacro)
@@ -115,4 +115,65 @@
     <origin xyz="0 0 0.185" rpy="0 0 0"/>
   </joint>
+  <link name="left_finger">
+    <visual>
+      <geometry><box size="0.02 0.05 0.1"/></geometry>
+      <material name="grey"><color rgba="0.5 0.5 0.5 1"/></material>
+    </visual>
+    <collision>
+      <geometry><box size="0.02 0.05 0.1"/></geometry>
+    </collision>
+    <inertial>
+      <mass value="0.1"/>
+      <inertia ixx="0.001" ixy="0" ixz="0" iyy="0.001" iyz="0" izz="0.001"/>
+    </inertial>
+  </link>
+  <!-- Gripper Right Finger -->
+  <link name="right_finger">
+    <visual>
+      <geometry><box size="0.02 0.05 0.1"/></geometry>
+      <material name="grey"/>
+    </visual>
+    <collision>
+      <geometry><box size="0.02 0.05 0.1"/></geometry>
+    </collision>
+    <inertial>
+      <mass value="0.1"/>
+      <inertia ixx="0.001" ixy="0" ixz="0" iyy="0.001" iyz="0" izz="0.001"/>
+    </inertial>
+  </link>
+  <joint name="gripper_left_joint" type="prismatic">
+    <parent link="tool0"/>
+    <child link="left_finger"/>
+    <origin xyz="0 0.05 0.05" rpy="0 0 0"/>
+    <axis xyz="0 1 0"/>
+    <limit effort="100" lower="-0.04" upper="0" velocity="0.2"/>
+  </joint>
+  <joint name="gripper_right_joint" type="prismatic">
+    <parent link="tool0"/>
+    <child link="right_finger"/>
+    <origin xyz="0 -0.05 0.05" rpy="0 0 0"/>
+    <axis xyz="0 1 0"/>
+    <limit effort="100" lower="0" upper="0.04" velocity="0.2"/>
+    <!-- In a real robot, this often mimics the left joint -->
+  </joint>
 </xacro:macro>
+  <gazebo reference="left_finger">
+    <mu1>1000.0</mu1>
+    <mu2>1000.0</mu2>
+    <kp>1000000.0</kp>
+    <kd>1.0</kd>
+    <material>Gazebo/Grey</material>
+  </gazebo>
+  <gazebo reference="right_finger">
+    <mu1>1000.0</mu1>
+    <mu2>1000.0</mu2>
+    <kp>1000000.0</kp>
+    <kd>1.0</kd>
+    <material>Gazebo/Grey</material>
+  </gazebo>
+  <gazebo>
+    <plugin filename="gz_ros2_control-system" name="gz_ros2_control::GazeboSimROS2ControlPlugin">
+      <parameters>$(find ros2_control_demo_example_7)/config/r6bot_controllers.yaml</parameters>
+    </plugin>
+  </gazebo>
 </robot>

Commit message: cube spawning & gazebo init

File: src/ros2_control_demos/example_7/description/ros2_control/r6bot.ros2_control.xacro (robot description, xacro)
@@ -1,8 +1,13 @@
 <?xml version="1.0"?>
 <robot xmlns:xacro="http://www.ros.org/wiki/xacro">
-  <xacro:macro name="r6bot_ros2_control" params="name">
+  <xacro:macro name="r6bot_ros2_control" params="name sim:=false">
     <ros2_control name="${name}" type="system">
       <hardware>
-        <plugin>mock_components/GenericSystem</plugin>
+        <xacro:if value="${sim}">
+          <plugin>gz_ros2_control/GazeboSimSystem</plugin>
+        </xacro:if>
+        <xacro:unless value="${sim}">
+          <plugin>mock_components/GenericSystem</plugin>
+        </xacro:unless>
       </hardware>
       <joint name="joint_1">

File: src/ros2_control_demos/example_7/description/urdf/r6bot.urdf.xacro (robot description, xacro)
@@ -1,11 +1,12 @@
 <?xml version="1.0"?>
-<robot xmlns:xacro="http://wiki.ros.org/xacro" name="r6bot">
+<robot xmlns:xacro="http://www.ros.org/wiki/xacro" name="r6bot">
+  <xacro:arg name="sim" default="false"/>
   <!-- Import r6bot macro -->
   <xacro:include filename="$(find ros2_control_demo_description)/r6bot/urdf/r6bot_description.urdf.xacro"/>
+  <!-- Import r6bot ros2_control description -->
+  <xacro:include filename="$(find ros2_control_demo_example_7)/ros2_control/r6bot.ros2_control.xacro"/>
   <!-- create link fixed to the "world" -->
   <link name="world"/>
   <xacro:r6bot_description/>
-  <!-- Import r6bot ros2_control description -->
-  <xacro:include filename="$(find ros2_control_demo_example_7)/ros2_control/r6bot.ros2_control.xacro" />
-  <xacro:r6bot_ros2_control name="r6bot"/>
+  <xacro:r6bot_ros2_control name="r6bot" sim="$(arg sim)"/>
 </robot>

File: src/ros2_control_demos/ros2_control_demo_description/r6bot/urdf/r6bot_description.urdf.xacro (robot description, xacro)
@@ -321,5 +321,5 @@
   <gazebo>
     <plugin filename="gz_ros2_control-system" name="gz_ros2_control::GazeboSimROS2ControlPlugin">
-      <parameters>$(find ros2_control_demo_example_7)/config/r6bot_controllers.yaml</parameters>
+      <parameters>$(find ros2_control_demo_example_7)/config/r6bot_controller.yaml</parameters>
     </plugin>
   </gazebo>
