Commit message: table improvments & drop-boxes added

File: src/ros2_control_demos/ros2_control_demo_description/r6bot/urdf/r6bot_description.urdf.xacro (robot description, xacro)
@@ -2,160 +2,308 @@
 <robot xmlns:xacro="http://www.ros.org/wiki/xacro">
   <xacro:macro name="r6bot_description">
-  <!-- helper macro -->
-  <xacro:include filename="$(find ros2_control_demo_description)/r6bot/urdf/inc/create_link.xacro"/>
-  <xacro:create_link
-      link_name="base_link"
-      xyz_offset="0 0 0"
-      rpy_offset="0 0 0"
-      mesh_package="ros2_control_demo_description/r6bot"
-      mesh_name="link_0"
-  />
-  <xacro:create_link
-      link_name="link_1"
-      xyz_offset="0 0 -0.182"
-      rpy_offset="0 0 0"
-      mesh_package="ros2_control_demo_description/r6bot"
-      mesh_name="link_1"
-  />
-  <xacro:create_link
-      link_name="link_2"
-      xyz_offset="0 0 -0.168"
-      rpy_offset="0 0 0"
-      mesh_package="ros2_control_demo_description/r6bot"
-      mesh_name="link_2"
-  />
-  <xacro:create_link
-      link_name="link_3"
-      xyz_offset="0 0 -0.144"
-      rpy_offset="0 0 0"
-      mesh_package="ros2_control_demo_description/r6bot"
-      mesh_name="link_3"
-  />
-  <xacro:create_link
-      link_name="link_4"
-      xyz_offset="0 0 0.077"
-      rpy_offset="0 0 0"
-      mesh_package="ros2_control_demo_description/r6bot"
-      mesh_name="link_4"
-  />
-  <xacro:create_link
-      link_name="link_5"
-      xyz_offset="0 0 0.113"
-      rpy_offset="0 0 0"
-      mesh_package="ros2_control_demo_description/r6bot"
-      mesh_name="link_5"
-  />
-  <xacro:create_link
-      link_name="link_6"
-      xyz_offset="0 0 0.086"
-      rpy_offset="0 0 0"
-      mesh_package="ros2_control_demo_description/r6bot"
-      mesh_name="link_6"
-  />
-  <link name="ft_frame"/>
-  <link name="tool0"/>
-  <!-- base_joint fixes base_link to the environment -->
-  <joint name="base_joint" type="fixed">
-    <parent link="world"/>
-    <child link="base_link"/>
-    <origin xyz="0 0 0" rpy="0 0 0"/>
-    <axis xyz="0 0 1"/>
-  </joint>
-  <!-- joints - main serial chain -->
-  <joint name="joint_1" type="revolute">
-    <parent link="base_link"/>
-    <child link="link_1"/>
-    <origin xyz="0 0 0.244" rpy="0 0 0"/>
-    <axis xyz="0 0 1"/>
-    <limit effort="1000.0" lower="${-pi}" upper="${pi}" velocity="2.5"/>
-  </joint>
-  <joint name="joint_2" type="revolute">
-    <parent link="link_1"/>
-    <child link="link_2"/>
-    <origin xyz="-0.27 0 0.0" rpy="${-pi/2} -${pi/2} ${pi/2}"/>
-    <axis xyz="0 0 1"/>
-    <limit effort="1000.0" lower="${-pi}" upper="${pi}" velocity="2.5"/>
-  </joint>
-  <joint name="joint_3" type="revolute">
-    <parent link="link_2"/>
-    <child link="link_3"/>
-    <origin xyz="0.686 0 -0.27" rpy="0 ${pi} ${pi+pi/2}"/>
-    <axis xyz="0 0 1"/>
-    <limit effort="1000.0" lower="${-pi}" upper="${pi}" velocity="2.5"/>
-  </joint>
-  <joint name="joint_4" type="revolute">
-    <parent link="link_3"/>
-    <child link="link_4"/>
-    <origin xyz="0.519 0 0" rpy="0 ${pi} ${pi}"/>
-    <axis xyz="0 0 1"/>
-    <limit effort="1000.0" lower="${-pi}" upper="${pi}" velocity="2.5"/>
-  </joint>
-  <joint name="joint_5" type="revolute">
-    <parent link="link_4"/>
-    <child link="link_5"/>
-    <origin xyz="0.0 0 0.188" rpy="${pi/2} ${pi} ${pi/2}"/>
-    <axis xyz="0 0 1"/>
-    <limit effort="1000.0" lower="${-pi}" upper="${pi}" velocity="2.5"/>
-  </joint>
-  <joint name="joint_6" type="revolute">
-    <parent link="link_5"/>
-    <child link="link_6"/>
-    <origin xyz="0.0 0 0.246" rpy="0 ${-pi/2} 0"/>
-    <axis xyz="0 0 1"/>
-    <limit effort="1000.0" lower="${-pi}" upper="${pi}" velocity="2.5"/>
-  </joint>
-  <joint name="joint-ft_frame" type="fixed">
-    <parent link="link_6"/>
-    <child link="ft_frame"/>
-    <origin xyz="0 0 0.086" rpy="0 0 0"/>
-  </joint>
-  <joint name="joint-tool" type="fixed">
-    <parent link="ft_frame"/>
-    <child link="tool0"/>
-    <origin xyz="0 0 0.185" rpy="0 0 0"/>
-  </joint>
-  <link name="left_finger">
-    <visual>
-      <geometry><box size="0.02 0.05 0.1"/></geometry>
-      <material name="grey"><color rgba="0.5 0.5 0.5 1"/></material>
-    </visual>
-    <collision>
-      <geometry><box size="0.02 0.05 0.1"/></geometry>
-    </collision>
-    <inertial>
-      <mass value="0.1"/>
-      <inertia ixx="0.001" ixy="0" ixz="0" iyy="0.001" iyz="0" izz="0.001"/>
-    </inertial>
-  </link>
-  <!-- Gripper Right Finger -->
-  <link name="right_finger">
-    <visual>
-      <geometry><box size="0.02 0.05 0.1"/></geometry>
-      <material name="grey"/>
-    </visual>
-    <collision>
-      <geometry><box size="0.02 0.05 0.1"/></geometry>
-    </collision>
-    <inertial>
-      <mass value="0.1"/>
-      <inertia ixx="0.001" ixy="0" ixz="0" iyy="0.001" iyz="0" izz="0.001"/>
-    </inertial>
-  </link>
-  <joint name="gripper_left_joint" type="prismatic">
-    <parent link="tool0"/>
-    <child link="left_finger"/>
-    <origin xyz="0 0.05 0.05" rpy="0 0 0"/>
-    <axis xyz="0 1 0"/>
-    <limit effort="100" lower="-0.04" upper="0" velocity="0.2"/>
-  </joint>
-  <joint name="gripper_right_joint" type="prismatic">
-    <parent link="tool0"/>
-    <child link="right_finger"/>
-    <origin xyz="0 -0.05 0.05" rpy="0 0 0"/>
-    <axis xyz="0 1 0"/>
-    <limit effort="100" lower="0" upper="0.04" velocity="0.2"/>
-    <!-- In a real robot, this often mimics the left joint -->
-  </joint>
-</xacro:macro>
+    <!-- helper macro -->
+    <xacro:include filename="$(find ros2_control_demo_description)/r6bot/urdf/inc/create_link.xacro"/>
+    <!-- ====== WORKSPACE TABLE ====== -->
+    <!-- Table Top (2.0m x 1.6m x 0.05m) -->
+    <link name="table">
+      <visual>
+        <geometry>
+          <box size="2.0 1.6 0.05"/>
+        </geometry>
+        <!-- The top surface is at Z=0.75, so the center of a 0.05m thick board is at 0.725 -->
+        <origin xyz="0 0 0.725" rpy="0 0 0"/>
+        <material name="table_wood">
+          <color rgba="0.72 0.53 0.34 1.0"/>
+        </material>
+      </visual>
+      <collision>
+        <geometry>
+          <box size="2.0 1.6 0.05"/>
+        </geometry>
+        <origin xyz="0 0 0.725" rpy="0 0 0"/>
+      </collision>
+      <inertial>
+        <mass value="50.0"/>
+        <origin xyz="0 0 0.725" rpy="0 0 0"/>
+        <inertia ixx="4.0" ixy="0" ixz="0" iyy="4.0" iyz="0" izz="4.0"/>
+      </inertial>
+    </link>
+    <!-- Fix table to world -->
+    <joint name="world_to_table" type="fixed">
+      <parent link="world"/>
+      <child link="table"/>
+      <origin xyz="0 0 0" rpy="0 0 0"/>
+    </joint>
+    <!-- Table Legs Macro -->
+    <xacro:macro name="table_leg" params="prefix x y">
+      <link name="${prefix}_leg">
+        <visual>
+          <geometry>
+            <cylinder radius="0.04" length="0.70"/>
+          </geometry>
+          <origin xyz="0 0 0.35" rpy="0 0 0"/>
+          <material name="leg_metal">
+            <color rgba="0.2 0.2 0.2 1.0"/>
+          </material>
+        </visual>
+        <collision>
+          <geometry>
+            <cylinder radius="0.04" length="0.70"/>
+          </geometry>
+          <origin xyz="0 0 0.35" rpy="0 0 0"/>
+        </collision>
+        <inertial>
+          <mass value="5.0"/>
+          <origin xyz="0 0 0.35" rpy="0 0 0"/>
+          <inertia ixx="0.1" ixy="0" ixz="0" iyy="0.1" iyz="0" izz="0.01"/>
+        </inertial>
+      </link>
+      <joint name="${prefix}_leg_joint" type="fixed">
+        <parent link="table"/>
+        <child link="${prefix}_leg"/>
+        <origin xyz="${x} ${y} 0" rpy="0 0 0"/>
+      </joint>
+    </xacro:macro>
+    <!-- Instantiate 4 Legs -->
+    <xacro:table_leg prefix="front_left" x="-0.9" y="0.7"/>
+    <xacro:table_leg prefix="front_right" x="0.9" y="0.7"/>
+    <xacro:table_leg prefix="back_left" x="-0.9" y="-0.7"/>
+    <xacro:table_leg prefix="back_right" x="0.9" y="-0.7"/>
+    <!-- Mount arm at back center edge of table -->
+    <joint name="base_joint" type="fixed">
+      <parent link="table"/>
+      <child link="base_link"/>
+      <origin xyz="0 -0.8 0.75" rpy="0 0 0"/>
+    </joint>
+    <!-- ====== SHELLED BINS ====== -->
+    <!-- Macro to create an open-top container (5 distinct collision boxes) -->
+    <xacro:macro name="shelled_bin" params="prefix color_name rgba x y">
+      <link name="${prefix}_bin">
+        <!-- Bottom Plate -->
+        <visual>
+          <origin xyz="0 0 0.01"/>
+          <geometry><box size="0.3 0.3 0.02"/></geometry>
+          <material name="${color_name}"><color rgba="${rgba}"/></material>
+        </visual>
+        <collision>
+          <origin xyz="0 0 0.01"/>
+          <geometry><box size="0.3 0.3 0.02"/></geometry>
+        </collision>
+        <!-- Front Wall -->
+        <visual>
+          <origin xyz="0 0.14 0.1"/>
+          <geometry><box size="0.3 0.02 0.2"/></geometry>
+          <material name="${color_name}"/>
+        </visual>
+        <collision>
+          <origin xyz="0 0.14 0.1"/>
+          <geometry><box size="0.3 0.02 0.2"/></geometry>
+        </collision>
+        <!-- Back Wall -->
+        <visual>
+          <origin xyz="0 -0.14 0.1"/>
+          <geometry><box size="0.3 0.02 0.2"/></geometry>
+          <material name="${color_name}"/>
+        </visual>
+        <collision>
+          <origin xyz="0 -0.14 0.1"/>
+          <geometry><box size="0.3 0.02 0.2"/></geometry>
+        </collision>
+        <!-- Left Wall -->
+        <visual>
+          <origin xyz="-0.14 0 0.1"/>
+          <geometry><box size="0.02 0.26 0.2"/></geometry>
+          <material name="${color_name}"/>
+        </visual>
+        <collision>
+          <origin xyz="-0.14 0 0.1"/>
+          <geometry><box size="0.02 0.26 0.2"/></geometry>
+        </collision>
+        <!-- Right Wall -->
+        <visual>
+          <origin xyz="0.14 0 0.1"/>
+          <geometry><box size="0.02 0.26 0.2"/></geometry>
+          <material name="${color_name}"/>
+        </visual>
+        <collision>
+          <origin xyz="0.14 0 0.1"/>
+          <geometry><box size="0.02 0.26 0.2"/></geometry>
+        </collision>
+        <inertial>
+          <mass value="1.5"/>
+          <origin xyz="0 0 0.1"/>
+          <inertia ixx="0.01" ixy="0" ixz="0" iyy="0.01" iyz="0" izz="0.01"/>
+        </inertial>
+      </link>
+      <joint name="${prefix}_bin_joint" type="fixed">
+        <parent link="table"/>
+        <child link="${prefix}_bin"/>
+        <!-- Placed perfectly on top of the table (Z=0.75) -->
+        <origin xyz="${x} ${y} 0.75" rpy="0 0 0"/>
+      </joint>
+    </xacro:macro>
+    <!-- Spawn the 3 bins hanging off the right edge of the table -->
+    <xacro:shelled_bin prefix="red" color_name="BinRed" rgba="0.8 0.1 0.1 1.0" x="1.15" y="-0.4"/>
+    <xacro:shelled_bin prefix="green" color_name="BinGreen" rgba="0.1 0.8 0.1 1.0" x="1.15" y="0.0"/>
+    <xacro:shelled_bin prefix="blue" color_name="BinBlue" rgba="0.1 0.1 0.8 1.0" x="1.15" y="0.4"/>
+    <!-- ====== ARM LINKS ====== -->
+    <xacro:create_link
+        link_name="base_link"
+        xyz_offset="0 0 0"
+        rpy_offset="0 0 0"
+        mesh_package="ros2_control_demo_description/r6bot"
+        mesh_name="link_0"
+    />
+    <xacro:create_link
+        link_name="link_1"
+        xyz_offset="0 0 -0.182"
+        rpy_offset="0 0 0"
+        mesh_package="ros2_control_demo_description/r6bot"
+        mesh_name="link_1"
+    />
+    <xacro:create_link
+        link_name="link_2"
+        xyz_offset="0 0 -0.168"
+        rpy_offset="0 0 0"
+        mesh_package="ros2_control_demo_description/r6bot"
+        mesh_name="link_2"
+    />
+    <xacro:create_link
+        link_name="link_3"
+        xyz_offset="0 0 -0.144"
+        rpy_offset="0 0 0"
+        mesh_package="ros2_control_demo_description/r6bot"
+        mesh_name="link_3"
+    />
+    <xacro:create_link
+        link_name="link_4"
+        xyz_offset="0 0 0.077"
+        rpy_offset="0 0 0"
+        mesh_package="ros2_control_demo_description/r6bot"
+        mesh_name="link_4"
+    />
+    <xacro:create_link
+        link_name="link_5"
+        xyz_offset="0 0 0.113"
+        rpy_offset="0 0 0"
+        mesh_package="ros2_control_demo_description/r6bot"
+        mesh_name="link_5"
+    />
+    <xacro:create_link
+        link_name="link_6"
+        xyz_offset="0 0 0.086"
+        rpy_offset="0 0 0"
+        mesh_package="ros2_control_demo_description/r6bot"
+        mesh_name="link_6"
+    />
+    <link name="ft_frame"/>
+    <link name="tool0"/>
+    <!-- ====== ARM JOINTS (serial chain) ====== -->
+    <joint name="joint_1" type="revolute">
+      <parent link="base_link"/>
+      <child link="link_1"/>
+      <origin xyz="0 0 0.244" rpy="0 0 0"/>
+      <axis xyz="0 0 1"/>
+      <limit effort="1000.0" lower="${-pi}" upper="${pi}" velocity="2.5"/>
+    </joint>
+    <joint name="joint_2" type="revolute">
+      <parent link="link_1"/>
+      <child link="link_2"/>
+      <origin xyz="-0.27 0 0.0" rpy="${-pi/2} -${pi/2} ${pi/2}"/>
+      <axis xyz="0 0 1"/>
+      <limit effort="1000.0" lower="${-pi}" upper="${pi}" velocity="2.5"/>
+    </joint>
+    <joint name="joint_3" type="revolute">
+      <parent link="link_2"/>
+      <child link="link_3"/>
+      <origin xyz="0.686 0 -0.27" rpy="0 ${pi} ${pi+pi/2}"/>
+      <axis xyz="0 0 1"/>
+      <limit effort="1000.0" lower="${-pi}" upper="${pi}" velocity="2.5"/>
+    </joint>
+    <joint name="joint_4" type="revolute">
+      <parent link="link_3"/>
+      <child link="link_4"/>
+      <origin xyz="0.519 0 0" rpy="0 ${pi} ${pi}"/>
+      <axis xyz="0 0 1"/>
+      <limit effort="1000.0" lower="${-pi}" upper="${pi}" velocity="2.5"/>
+    </joint>
+    <joint name="joint_5" type="revolute">
+      <parent link="link_4"/>
+      <child link="link_5"/>
+      <origin xyz="0.0 0 0.188" rpy="${pi/2} ${pi} ${pi/2}"/>
+      <axis xyz="0 0 1"/>
+      <limit effort="1000.0" lower="${-pi}" upper="${pi}" velocity="2.5"/>
+    </joint>
+    <joint name="joint_6" type="revolute">
+      <parent link="link_5"/>
+      <child link="link_6"/>
+      <origin xyz="0.0 0 0.246" rpy="0 ${-pi/2} 0"/>
+      <axis xyz="0 0 1"/>
+      <limit effort="1000.0" lower="${-pi}" upper="${pi}" velocity="2.5"/>
+    </joint>
+    <joint name="joint-ft_frame" type="fixed">
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
Commit message: added bigger bins

File: src/ros2_control_demos/ros2_control_demo_description/r6bot/urdf/r6bot_description.urdf.xacro (robot description, xacro)
@@ -78,59 +78,59 @@
     <!-- ====== SHELLED BINS ====== -->
     <!-- Macro to create an open-top container (5 distinct collision boxes) -->
-    <xacro:macro name="shelled_bin" params="prefix color_name rgba x y">
+<xacro:macro name="shelled_bin" params="prefix color_name rgba x y">
       <link name="${prefix}_bin">
         <!-- Bottom Plate -->
         <visual>
           <origin xyz="0 0 0.01"/>
-          <geometry><box size="0.3 0.3 0.02"/></geometry>
+          <geometry><box size="0.38 0.38 0.02"/></geometry>
           <material name="${color_name}"><color rgba="${rgba}"/></material>
         </visual>
         <collision>
           <origin xyz="0 0 0.01"/>
-          <geometry><box size="0.3 0.3 0.02"/></geometry>
+          <geometry><box size="0.38 0.38 0.02"/></geometry>
         </collision>
         <!-- Front Wall -->
         <visual>
-          <origin xyz="0 0.14 0.1"/>
-          <geometry><box size="0.3 0.02 0.2"/></geometry>
+          <origin xyz="0 0.18 0.17"/>
+          <geometry><box size="0.38 0.02 0.30"/></geometry>
           <material name="${color_name}"/>
         </visual>
         <collision>
-          <origin xyz="0 0.14 0.1"/>
-          <geometry><box size="0.3 0.02 0.2"/></geometry>
+          <origin xyz="0 0.18 0.17"/>
+          <geometry><box size="0.38 0.02 0.30"/></geometry>
         </collision>
         <!-- Back Wall -->
         <visual>
-          <origin xyz="0 -0.14 0.1"/>
-          <geometry><box size="0.3 0.02 0.2"/></geometry>
+          <origin xyz="0 -0.18 0.17"/>
+          <geometry><box size="0.38 0.02 0.30"/></geometry>
           <material name="${color_name}"/>
         </visual>
         <collision>
-          <origin xyz="0 -0.14 0.1"/>
-          <geometry><box size="0.3 0.02 0.2"/></geometry>
+          <origin xyz="0 -0.18 0.17"/>
+          <geometry><box size="0.38 0.02 0.30"/></geometry>
         </collision>
         <!-- Left Wall -->
         <visual>
-          <origin xyz="-0.14 0 0.1"/>
-          <geometry><box size="0.02 0.26 0.2"/></geometry>
+          <origin xyz="-0.18 0 0.17"/>
+          <geometry><box size="0.02 0.34 0.30"/></geometry>
           <material name="${color_name}"/>
         </visual>
         <collision>
-          <origin xyz="-0.14 0 0.1"/>
-          <geometry><box size="0.02 0.26 0.2"/></geometry>
+          <origin xyz="-0.18 0 0.17"/>
+          <geometry><box size="0.02 0.34 0.30"/></geometry>
         </collision>
         <!-- Right Wall -->
         <visual>
-          <origin xyz="0.14 0 0.1"/>
-          <geometry><box size="0.02 0.26 0.2"/></geometry>
+          <origin xyz="0.18 0 0.17"/>
+          <geometry><box size="0.02 0.34 0.30"/></geometry>
           <material name="${color_name}"/>
         </visual>
         <collision>
-          <origin xyz="0.14 0 0.1"/>
-          <geometry><box size="0.02 0.26 0.2"/></geometry>
+          <origin xyz="0.18 0 0.17"/>
+          <geometry><box size="0.02 0.34 0.30"/></geometry>
         </collision>
         <inertial>
           <mass value="1.5"/>
-          <origin xyz="0 0 0.1"/>
+          <origin xyz="0 0 0.17"/>
           <inertia ixx="0.01" ixy="0" ixz="0" iyy="0.01" iyz="0" izz="0.01"/>
         </inertial>
@@ -139,12 +139,11 @@
         <parent link="table"/>
         <child link="${prefix}_bin"/>
-        <!-- Placed perfectly on top of the table (Z=0.75) -->
         <origin xyz="${x} ${y} 0.75" rpy="0 0 0"/>
       </joint>
     </xacro:macro>
     <!-- Spawn the 3 bins hanging off the right edge of the table -->
-    <xacro:shelled_bin prefix="red" color_name="BinRed" rgba="0.8 0.1 0.1 1.0" x="1.15" y="-0.4"/>
-    <xacro:shelled_bin prefix="green" color_name="BinGreen" rgba="0.1 0.8 0.1 1.0" x="1.15" y="0.0"/>
-    <xacro:shelled_bin prefix="blue" color_name="BinBlue" rgba="0.1 0.1 0.8 1.0" x="1.15" y="0.4"/>
+    <xacro:shelled_bin prefix="red" color_name="BinRed" rgba="0.8 0.1 0.1 1.0" x="1.05" y="-0.4"/>
+    <xacro:shelled_bin prefix="green" color_name="BinGreen" rgba="0.1 0.8 0.1 1.0" x="1.05" y="0.0"/>
+    <xacro:shelled_bin prefix="blue" color_name="BinBlue" rgba="0.1 0.1 0.8 1.0" x="1.05" y="0.4"/>
     <!-- ====== ARM LINKS ====== -->
     <xacro:create_link

Commit message: basic camara implementaion

File: src/ros2_control_demos/ros2_control_demo_description/r6bot/urdf/r6bot_description.urdf.xacro (robot description, xacro)
@@ -292,4 +292,24 @@
       <limit effort="100" lower="0" upper="0.04" velocity="0.2"/>
     </joint>
+    <!-- ====== OVERHEAD CAMERA ====== -->
+    <link name="camera_link">
+      <visual>
+        <geometry><box size="0.05 0.05 0.05"/></geometry>
+        <material name="camera_black">
+          <color rgba="0.1 0.1 0.1 1.0"/>
+        </material>
+      </visual>
+      <inertial>
+        <mass value="0.1"/>
+        <inertia ixx="0.0001" ixy="0" ixz="0"
+                 iyy="0.0001" iyz="0" izz="0.0001"/>
+      </inertial>
+    </link>
+    <joint name="camera_joint" type="fixed">
+      <parent link="table"/>
+      <child link="camera_link"/>
+      <!-- 1.05m above table surface, centered over workspace -->
+      <origin xyz="0.1 0.2 3.1" rpy="0 1.5708 0"/>
+    </joint>
   </xacro:macro>
   <!-- ====== GAZEBO PROPERTIES ====== -->
@@ -324,3 +344,30 @@
     </plugin>
   </gazebo>
+<!-- Overhead RGBD Camera -->
+  <gazebo reference="camera_link">
+    <sensor name="rgbd_camera" type="rgbd_camera">
+      <camera>
+        <horizontal_fov>1.3</horizontal_fov>
+        <image>
+          <width>640</width>
+          <height>480</height>
+          <format>R8G8B8</format>
+        </image>
+        <clip>
+          <near>0.1</near>
+          <far>5.0</far>
+        </clip>
+        <depth_camera>
+          <clip>
+            <near>0.1</near>
+            <far>5.0</far>
+          </clip>
+        </depth_camera>
+      </camera>
+      <always_on>1</always_on>
+      <update_rate>15</update_rate>
+      <visualize>true</visualize>
+      <topic>overhead_camera</topic>
+    </sensor>
+  </gazebo>
 </robot>

Commit message: final commit

File: src/ros2_control_demos/ros2_control_demo_description/r6bot/urdf/r6bot_description.urdf.xacro (robot description, xacro)
@@ -283,5 +283,5 @@
       <origin xyz="0 0.05 0.05" rpy="0 0 0"/>
       <axis xyz="0 1 0"/>
-      <limit effort="100" lower="-0.04" upper="0" velocity="0.2"/>
+      <limit effort="100" lower="-0.06" upper="0" velocity="0.2"/>
     </joint>
     <joint name="gripper_right_joint" type="prismatic">
@@ -290,5 +290,5 @@
       <origin xyz="0 -0.05 0.05" rpy="0 0 0"/>
       <axis xyz="0 1 0"/>
-      <limit effort="100" lower="0" upper="0.04" velocity="0.2"/>
+      <limit effort="100" lower="0" upper="0.06" velocity="0.2"/>
     </joint>
     <!-- ====== OVERHEAD CAMERA ====== -->
